File: hardware/kicad/ildagenerator.sch (KiCad schematic (older format))
At the start: 5 parts, among them P7 CONN_6, P8 CONN_4, U1 LTC2656BIFE-L16

Commit message: onboard power dc/dc
Parts:
- added MOV13: 5.6V, Resistors_SMD:R_1206_HandSoldering, symbol VR
- added U5: NMA0509SC, footprints:NMA_5V_12V_15V_Series, symbol NMA0509SC
- P7: footprint (none) -> Pin_Headers:Pin_Header_Straight_1x06; symbol CONN_6 -> CONN_01X06
- P8: footprint (none) -> Pin_Headers:Pin_Header_Straight_1x02; symbol CONN_4 -> CONN_01X02
Connections:
- net +15V: now also U5.6 (+Vout); no longer P8.3 (P3)
- net +5V: now also MOV13.1, U5.1 (+Vin)
- net -15V: now also U5.4 (-Vout); no longer P8.4 (P4)
- net GND: now also MOV13.2, U5.2 (-Vin), U5.5 (0V)
Other:
- moved on the sheet: P7
Changed lines of the file:
@@
 LIBS:contrib
 LIBS:valves
+LIBS:dc_dc
 LIBS:ildagenerator-cache
 EELAYER 25 0
@@
 	4900 4050 4900 4200
 Wire Wire Line
-	4700 4200 4700 4100
-Wire Wire Line
 	3800 4200 3800 4100
 Wire Wire Line
@@
 Wire Wire Line
 	2600 3000 2800 3000
-Wire Wire Line
-	4600 4200 4600 4100
-Wire Wire Line
-	4800 4200 4800 4100
-$Comp
-L GND-RESCUE-ildagenerator #PWR8
+$Comp
+L GND-RESCUE-ildagenerator #PWR7
 U 1 1 53E63A9F
-P 5000 4050
-F 0 "#PWR8" H 5000 4050 30  0001 C CNN
-F 1 "GND" H 5000 3980 30  0001 C CNN
-F 2 "" H 5000 4050 60  0001 C CNN
-F 3 "" H 5000 4050 60  0001 C CNN
-	1    5000 4050
-	1    0    0    -1
-$EndComp
-$Comp
-L +5V #PWR7
+P 5000 4100
+F 0 "#PWR7" H 5000 4100 30  0001 C CNN
+F 1 "GND" H 5000 4030 30  0001 C CNN
+F 2 "" H 5000 4100 60  0001 C CNN
+F 3 "" H 5000 4100 60  0001 C CNN
+	1    5000 4100
+	1    0    0    -1
+$EndComp
+$Comp
+L +5V #PWR6
 U 1 1 53E63A98
-P 4800 4100
-F 0 "#PWR7" H 4800 4190 20  0001 C CNN
-F 1 "+5V" H 4800 4190 30  0000 C CNN
-F 2 "" H 4800 4100 60  0001 C CNN
-F 3 "" H 4800 4100 60  0001 C CNN
-	1    4800 4100
-	1    0    0    -1
-$EndComp
-$Comp
-L +15V #PWR6
+P 4800 3950
+F 0 "#PWR6" H 4800 4040 20  0001 C CNN
+F 1 "+5V" H 4800 4040 30  0000 C CNN
+F 2 "" H 4800 3950 60  0001 C CNN
+F 3 "" H 4800 3950 60  0001 C CNN
+	1    4800 3950
+	1    0    0    -1
+$EndComp
+$Comp
+L +15V #PWR11
 U 1 1 53E63A91
-P 4700 4100
-F 0 "#PWR6" H 4700 4050 20  0001 C CNN
-F 1 "+15V" H 4700 4200 30  0000 C CNN
-F 2 "" H 4700 4100 60  0001 C CNN
-F 3 "" H 4700 4100 60  0001 C CNN
-	1    4700 4100
-	1    0    0    -1
-$EndComp
-$Comp
-L -15V #PWR3
+P 6300 3550
+F 0 "#PWR11" H 6300 3500 20  0001 C CNN
+F 1 "+15V" H 6300 3650 30  0000 C CNN
+F 2 "" H 6300 3550 60  0001 C CNN
+F 3 "" H 6300 3550 60  0001 C CNN
+	1    6300 3550
+	1    0    0    -1
+$EndComp
+$Comp
+L -15V #PWR12
 U 1 1 53E63A8A
-P 4600 4100
-F 0 "#PWR3" H 4600 4230 20  0001 C CNN
-F 1 "-15V" H 4600 4200 30  0000 C CNN
-F 2 "" H 4600 4100 60  0001 C CNN
-F 3 "" H 4600 4100 60  0001 C CNN
-	1    4600 4100
-	1    0    0    -1
-$EndComp
-$Comp
-L CONN_4 P8
+P 6300 3850
+F 0 "#PWR12" H 6300 3980 20  0001 C CNN
+F 1 "-15V" H 6300 3950 30  0000 C CNN
+F 2 "" H 6300 3850 60  0001 C CNN
+F 3 "" H 6300 3850 60  0001 C CNN
+	1    6300 3850
+	1    0    0    -1
+$EndComp
+$Comp
+L CONN_01X02 P8
 U 1 1 53E639B6
-P 4750 4550
-F 0 "P8" V 4700 4550 50  0000 C CNN
-F 1 "CONN_4" V 4800 4550 50  0000 C CNN
-F 2 "" H 4750 4550 60  0001 C CNN
-F 3 "" H 4750 4550 60  0001 C CNN
-	1    4750 4550
+P 4850 4400
+F 0 "P8" V 4800 4400 50  0000 C CNN
+F 1 "CONN_4" V 4900 4400 50  0000 C CNN
+F 2 "Pin_Headers:Pin_Header_Straight_1x02" H 4850 4400 60  0001 C CNN
+F 3 "" H 4850 4400 60  0001 C CNN
+	1    4850 4400
 	0    1    1    0
 $EndComp
@@
 	1    3950 4200
 	1    0    0    -1
-$EndComp
-$Comp
-L CONN_6 P7
-U 1 1 53E5FC4C
-P 3550 4550
-F 0 "P7" V 3500 4550 60  0000 C CNN
-F 1 "CONN_6" V 3600 4550 60  0000 C CNN
-F 2 "" H 3550 4550 60  0001 C CNN
-F 3 "" H 3550 4550 60  0001 C CNN
-	1    3550 4550
-	0    1    1    0
 $EndComp
 $Comp
@@
 $EndComp
 $Comp
-L GND-RESCUE-ildagenerator #PWR9
+L GND-RESCUE-ildagenerator #PWR10
 U 1 1 53E2274C
 P 5200 3050
-F 0 "#PWR9" H 5200 3050 30  0001 C CNN
+F 0 "#PWR10" H 5200 3050 30  0001 C CNN
 F 1 "GND" H 5200 2980 30  0001 C CNN
 F 2 "" H 5200 3050 60  0001 C CNN
@@
 	1    0    0    -1
 $EndComp
+$Comp
+L NMA0509SC U5
+U 1 1 55E4611A
+P 5750 3700
+F 0 "U5" H 5750 3400 60  0000 C CNN
+F 1 "NMA0509SC" H 5750 4000 60  0000 C CNN
+F 2 "footprints:NMA_5V_12V_15V_Series" H 5750 3700 60  0001 C CNN
+F 3 "http://power.murata.com/data/power/ncl/kdc_nms.pdf" H 5750 3700 60  0001 C CNN
+	1    5750 3700
+	1    0    0    -1
+$EndComp
+Wire Wire Line
+	5000 4050 5000 4100
+$Comp
+L +5V #PWR8
+U 1 1 55E47078
+P 5150 3500
+F 0 "#PWR8" H 5150 3590 20  0001 C CNN
+F 1 "+5V" H 5150 3590 30  0000 C CNN
+F 2 "" H 5150 3500 60  0001 C CNN
+F 3 "" H 5150 3500 60  0001 C CNN
+	1    5150 3500
+	1    0    0    -1
+$EndComp
+Wire Wire Line
+	5150 3500 5150 3550
+Wire Wire Line
+	5150 3550 5250 3550
+$Comp
+L GND-RESCUE-ildagenerator #PWR9
+U 1 1 55E47142
+P 5150 3900
+F 0 "#PWR9" H 5150 3900 30  0001 C CNN
+F 1 "GND" H 5150 3830 30  0001 C CNN
+F 2 "" H 5150 3900 60  0001 C CNN
+F 3 "" H 5150 3900 60  0001 C CNN
+	1    5150 3900
+	1    0    0    -1
+$EndComp
+Wire Wire Line
+	5250 3850 5150 3850
+Wire Wire Line
+	5150 3850 5150 3900
+$Comp
+L GND-RESCUE-ildagenerator #PWR13
+U 1 1 55E476F0
+P 6450 3750
+F 0 "#PWR13" H 6450 3750 30  0001 C CNN
+F 1 "GND" H 6450 3680 30  0001 C CNN
+F 2 "" H 6450 3750 60  0001 C CNN
+F 3 "" H 6450 3750 60  0001 C CNN
+	1    6450 3750
+	1    0    0    -1
+$EndComp
+Wire Wire Line
+	6250 3850 6300 3850
+Wire Wire Line
+	6250 3550 6300 3550
+Wire Wire Line
+	6250 3700 6450 3700
+Wire Wire Line
+	6450 3700 6450 3750
+$Comp
+L CONN_01X06 P7
+U 1 1 53E5FC4C
+P 3550 4400
+F 0 "P7" V 3500 4400 60  0000 C CNN
+F 1 "CONN_6" V 3600 4400 60  0000 C CNN
+F 2 "Pin_Headers:Pin_Header_Straight_1x06" H 3550 4400 60  0001 C CNN
+F 3 "" H 3550 4400 60  0001 C CNN
+	1    3550 4400
+	0    1    1    0
+$EndComp
+$Comp
+L VR MOV13
+U 1 1 55E49EC4
+P 4550 4050
+F 0 "MOV13" V 4610 4004 50  0000 C TNN
+F 1 "5.6V" V 4550 4050 50  0000 C CNN
+F 2 "Resistors_SMD:R_1206_HandSoldering" H 4550 4050 60  0001 C CNN
+F 3 "http://cdn-reichelt.de/documents/datenblatt/B400/VC%201206_Serie.pdf" H 4550 4050 60  0001 C CNN
+	1    4550 4050
+	0    1    1    0
+$EndComp
+Wire Wire Line
+	4800 3950 4800 4200
+Connection ~ 4800 4050
+Wire Wire Line
+	4300 4050 4300 4150
+$Comp
+L GND-RESCUE-ildagenerator #PWR3
+U 1 1 55E4A459
+P 4300 4150
+F 0 "#PWR3" H 4300 4150 30  0001 C CNN
+F 1 "GND" H 4300 4080 30  0001 C CNN
+F 2 "" H 4300 4150 60  0001 C CNN
+F 3 "" H 4300 4150 60  0001 C CNN
+	1    4300 4150
+	1    0    0    -1
+$EndComp
